File: plumber.kicad_pcb (KiCad board)
At the start: 2 copper layers, 60 x 40 mm, 99 parts, among them IC1 MP2451DT-LF-Z, J1 Conn_01x03, J2 Conn_01x03, J3 Conn_01x03, J4 Conn_01x03, J5 Conn_01x02, J6 Conn_01x02, J7 Conn_01x02, J8 Conn_01x02, J9 Conn_01x02, K1 ADW1103HLW, K2 ADW1103HLW, K3 ADW1103HLW, K4 ADW1103HLW, Q1 Si2319CDS, Q10 2N7002, Q11 Si2319CDS, Q12 2N7002, Q13 Si2319CDS, Q14 2N7002, Q15 Si2319CDS, Q16 2N7002, Q2 2N7002, Q3 Si2319CDS, Q4 2N7002, Q5 Si2319CDS, Q6 2N7002, Q7 Si2319CDS, Q8 2N7002, Q9 Si2319CDS, U1 ESP-12F

Commit message: hardware v1
Parts:
- removed BT1: 4 x AA(A), Connector_PinHeader_2.54mm:PinHeader_1x02_P2.54mm_Vertical
- removed D1, D10, D11, D12, D13, D14, D15, D16, D17, D18, D2, D3, D4, D5, D6, D7, D8, D9: D_Schottky, Diode_SMD:D_SOD-123
- removed the H2 at (399.7, 111.1)
- removed IC1: MP2451DT-LF-Z, SamacSys_Parts:SOT95P280X145-6N
- removed the J1 at (295.8, 59.9)
- removed J3: Conn_01x03, Connector_Harwin:Harwin_M20-89003xx_1x03_P2.54mm_Horizontal
- removed the J5 at (230.2, 63.8)
- removed the J8 at (278.5, 61.5)
- removed L1: 3.3u, Inductor_SMD:L_Bourns-SRN4018
- removed Q10, Q12, Q14, Q16, Q6, Q8: 2N7002, Package_TO_SOT_SMD:SOT-23
- removed Q11, Q13, Q15, Q5, Q7, Q9: Si2319CDS, Package_TO_SOT_SMD:SOT-23
- removed the R12 at (381.0, 141.6)
- removed the R17 at (402.4, 123.2)
- removed R19, R20, R21, R30, R31, R32, R33: 4.3, Resistor_SMD:R_0603_1608Metric
- removed R22, R24, R26, R28, R34, R36: 10k, Resistor_SMD:R_0402_1005Metric
- removed R23, R25, R27, R29, R35, R37: NC, Resistor_SMD:R_0402_1005Metric
- removed the R5 at (330.0, 149.7)
- added J10: Conn_01x02, TerminalBlock_Phoenix:TerminalBlock_Phoenix_MKDS-1,5-2_1x02_P5.00mm_Horizontal, F.Cu at (145.8, 66.5)
- added J11: Conn_01x02, TerminalBlock_Phoenix:TerminalBlock_Phoenix_MKDS-1,5-2_1x02_P5.00mm_Horizontal, F.Cu at (184.8, 66.5)
- added J12: Jack-DC, Connector_BarrelJack:BarrelJack_Horizontal, F.Cu at (131.8, 66.7)
- added J13: USB_B_Mini, Connector_USB:USB_Micro-B_Molex-105017-0001, F.Cu at (121.7, 66.4)
- added J2: Conn_01x03, Connector_PinSocket_2.54mm:PinSocket_1x03_P2.54mm_Vertical, F.Cu at (168.8, 95.0)
- added J6: Conn_01x03, Connector_PinSocket_2.54mm:PinSocket_1x03_P2.54mm_Vertical, F.Cu at (155.8, 95.0)
- added J9: Conn_01x03, Connector_PinSocket_2.54mm:PinSocket_1x03_P2.54mm_Vertical, F.Cu at (142.8, 95.0)
- added R4: 20k, Resistor_SMD:R_0603_1608Metric_Pad0.98x0.95mm_HandSolder, F.Cu at (173.0, 98.0)
- added R6: 10k, Resistor_SMD:R_0603_1608Metric_Pad0.98x0.95mm_HandSolder, F.Cu at (147.4, 107.0)
- added R9: 10k, Resistor_SMD:R_0603_1608Metric_Pad0.98x0.95mm_HandSolder, F.Cu at (178.0, 98.0)
- added U2: LM1117-3.3, Package_TO_SOT_SMD:SOT-223-3_TabPin2, F.Cu at (127.7, 87.2)
- added U3: LM1117-3.3, Package_TO_SOT_SMD:SOT-223-3_TabPin2, F.Cu at (124.5, 110.0)
- C1: footprint Capacitor_SMD:C_0402_1005Metric -> Capacitor_SMD:C_0603_1608Metric_Pad1.08x0.95mm_HandSolder
- C2: value 10u/10V -> 10u/16V; footprint Capacitor_SMD:C_0603_1608Metric -> Capacitor_THT:CP_Radial_D8.0mm_P3.50mm
- C3: value 33p -> 10u/16V; footprint Capacitor_SMD:C_0402_1005Metric -> Capacitor_THT:CP_Radial_D8.0mm_P3.50mm
- C4: value 100n -> 10u/16V; footprint Capacitor_SMD:C_0402_1005Metric -> Capacitor_THT:CP_Radial_D8.0mm_P3.50mm
- C5: value 4.7u/36V -> 100n/6.3V; footprint Capacitor_SMD:C_1206_3216Metric -> Capacitor_SMD:C_0603_1608Metric_Pad1.08x0.95mm_HandSolder
- C6: value 10u/6.3V -> 100n/6.3V; footprint Capacitor_SMD:C_0402_1005Metric -> Capacitor_SMD:C_0603_1608Metric_Pad1.08x0.95mm_HandSolder
- FLASH1, RESET1: footprint Button_Switch_SMD:SW_SPST_EVQP7A -> Button_Switch_SMD:SW_SPST_EVQPE1
- J4: footprint Connector_Harwin:Harwin_M20-89003xx_1x03_P2.54mm_Horizontal -> Connector_PinSocket_2.54mm:PinSocket_1x03_P2.54mm_Vertical
- J7: value Conn_01x02 -> Conn_01x04; footprint TerminalBlock_Phoenix:TerminalBlock_Phoenix_MKDS-1,5-2_1x02_P5.00mm_Horizontal -> Connector_PinSocket_2.54mm:PinSocket_1x04_P2.54mm_Vertical
- J8: renamed from J2; footprint Connector_Harwin:Harwin_M20-89003xx_1x03_P2.54mm_Horizontal -> Connector_PinSocket_2.54mm:PinSocket_1x03_P2.54mm_Vertical
- K1, K4: value ADW1103HLW -> 8-1419128-1; footprint SamacSys_Parts:ADW1103HLW -> SamacSys_Parts:814191281
- K2: renamed from K3; value ADW1103HLW -> 8-1419128-1; footprint SamacSys_Parts:ADW1103HLW -> SamacSys_Parts:814191281
- K3: renamed from K2; value ADW1103HLW -> 8-1419128-1; footprint SamacSys_Parts:ADW1103HLW -> SamacSys_Parts:814191281
- Q1, Q3: value Si2319CDS -> 2N7002
- R1: value 300k -> 10k; footprint Resistor_SMD:R_0402_1005Metric -> Resistor_SMD:R_0603_1608Metric_Pad0.98x0.95mm_HandSolder
- R10, R11, R16, R2, R8: footprint Resistor_SMD:R_0402_1005Metric -> Resistor_SMD:R_0603_1608Metric_Pad0.98x0.95mm_HandSolder
- R12: renamed from R6; footprint Resistor_SMD:R_0402_1005Metric -> Resistor_SMD:R_0603_1608Metric_Pad0.98x0.95mm_HandSolder
- R13: value 0 -> 20k; footprint Resistor_SMD:R_0402_1005Metric -> Resistor_SMD:R_0603_1608Metric_Pad0.98x0.95mm_HandSolder
- R14: value 10k -> 20k; footprint Resistor_SMD:R_0402_1005Metric -> Resistor_SMD:R_0603_1608Metric_Pad0.98x0.95mm_HandSolder
- R15: value NC -> 10k; footprint Resistor_SMD:R_0402_1005Metric -> Resistor_SMD:R_0603_1608Metric_Pad0.98x0.95mm_HandSolder
- R17: renamed from R9; footprint Resistor_SMD:R_0402_1005Metric -> Resistor_SMD:R_0603_1608Metric_Pad0.98x0.95mm_HandSolder
- R18: value 4.3 -> 0; footprint Resistor_SMD:R_0603_1608Metric -> Resistor_SMD:R_0603_1608Metric_Pad0.98x0.95mm_HandSolder
- R3: value 33k -> 10k; footprint Resistor_SMD:R_0402_1005Metric -> Resistor_SMD:R_0603_1608Metric_Pad0.98x0.95mm_HandSolder
- R5: renamed from R4; footprint Resistor_SMD:R_0402_1005Metric -> Resistor_SMD:R_0603_1608Metric_Pad0.98x0.95mm_HandSolder
- R7: value 47k -> 20k; footprint Resistor_SMD:R_0402_1005Metric -> Resistor_SMD:R_0603_1608Metric_Pad0.98x0.95mm_HandSolder
- moved R18 324.7 mm to (124.4, 72.4), turned to 180 degrees
- moved R15 297.0 mm to (139.0, 98.0)
- moved R14 292.7 mm to (147.1, 98.0)
- moved C3 274.8 mm to (125.5, 78.1), turned to 180 degrees
- moved Q1 273.6 mm to (165.0, 95.0), turned to 180 degrees
- moved C4 272.1 mm to (133.3, 113.7), turned to 90 degrees
- moved Q2 265.9 mm to (178.0, 95.0), turned to 180 degrees
- moved C5 260.0 mm to (123.1, 89.9), turned to 270 degrees
- moved C6 257.3 mm to (129.1, 107.3), turned to 90 degrees
- moved R10 254.5 mm to (156.0, 98.0)
- moved C2 244.9 mm to (130.7, 78.2)
- moved Q3 239.7 mm to (139.0, 95.0), turned to 180 degrees
- moved R8 239.6 mm to (165.0, 98.0)
- moved R11 238.5 mm to (143.0, 98.0)
- moved R13 231.1 mm to (160.1, 98.0)
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- renumbered H3 to H2, J6 to J1, J9 to J5
Connections:
- C2 pad 1: Net-(BT1-Pad1) -> VCC
- C3 pad 1: Net-(C3-Pad1) -> +5V
- C4 pad 1: Net-(C4-Pad1) -> +3V3
- C4 pad 2: Net-(C4-Pad2) -> GND
- C5 pad 1: VCC -> +5V
- J1 pad 1: AC_N -> Net-(J1-Pad1)
- J1 pad 2: Net-(J6-Pad2) -> Net-(J1-Pad2)
- J4 pad 1: +3V3 -> +5V
- J4 pad 2: RX -> Net-(J4-Pad2)
- J5 pad 1: AC_N -> Net-(J5-Pad1)
- J5 pad 2: Net-(J9-Pad2) -> Net-(J5-Pad2)
- J7 pad 1: AC_N -> +3V3
- J7 pad 2: Net-(J7-Pad2) -> TX
- J8 pad 2: GPIO0 -> GPIO2
- K1 pad 1: Net-(D2-Pad2) -> +5V
- K1 pad 3: Net-(J6-Pad2) -> Net-(K1-Pad3)
- K2 pad 1: Net-(D10-Pad2) -> +5V
- K2 pad 3: Net-(J8-Pad2) -> Net-(K2-Pad3)
- K3 pad 1: Net-(D4-Pad2) -> +5V
- K3 pad 3: Net-(J7-Pad2) -> Net-(K3-Pad3)
- K4 pad 1: Net-(D12-Pad2) -> +5V
- K4 pad 3: Net-(J9-Pad2) -> Net-(K4-Pad3)
- Q1 pad 1: GPIO12 -> GPIO10
- Q1 pad 2: Vdrive -> GND
- Q1 pad 3: Net-(Q1-Pad3) -> Net-(K1-Pad3)
- Q2 pad 1: GPIO12 -> GPIO13
- Q2 pad 3: Net-(D2-Pad2) -> Net-(K2-Pad3)
- Q3 pad 1: GPIO5 -> GPIO15
- Q3 pad 2: Vdrive -> GND
- Q3 pad 3: Net-(Q3-Pad3) -> Net-(K3-Pad3)
- Q4 pad 3: Net-(D4-Pad2) -> Net-(K4-Pad3)
- R1 pad 1: VCC -> Net-(J2-Pad2)
- R1 pad 2: ADC -> GPIO9
- R10 pad 1: +3V3 -> Net-(J6-Pad2)
- R10 pad 2: GPIO2 -> GPIO14
- R11 pad 1: GND -> Net-(J9-Pad2)
- R11 pad 2: GPIO15 -> GPIO4
- R13 pad 1: Vdrive -> GPIO14
- R13 pad 2: VCC -> GND
- R14 pad 1: Vdrive -> GPIO4
- R14 pad 2: GPIO12 -> GND
- R15 pad 2: GPIO12 -> GPIO15
- R16 pad 1: Vdrive -> GND
- R18 pad 1: Net-(Q1-Pad3) -> VCC
- R18 pad 2: Net-(D2-Pad2) -> +5V
- R2 pad 1: ADC -> +3V3
- R2 pad 2: GND -> GPIO2
- R3 pad 1: Net-(C3-Pad1) -> Net-(J4-Pad2)
- R3 pad 2: +3V3 -> GPIO12
- R7 pad 1: Net-(IC1-Pad4) -> GPIO12
- R7 pad 2: VCC -> GND
- R8 pad 1: +3V3 -> GND
- R8 pad 2: GPIO0 -> GPIO10
- U1 pad 10: Net-(U1-Pad10) -> (no net)
- U1 pad 13: Net-(U1-Pad13) -> (no net)
- U1 pad 14: Net-(U1-Pad14) -> (no net)
- U1 pad 2: ADC -> (no net)
- U1 pad 9: Net-(U1-Pad9) -> (no net)
Routing:
- net +5V: track 0.00 -> 156.6 mm
- net +3V3: track 0.00 -> 118.6 mm
- net VCC: track 0.00 -> 30.4 mm
- net GPIO4: track 0.00 -> 29.6 mm
- net GPIO2: track 0.00 -> 27.7 mm
- net GPIO5: track 0.00 -> 25.8 mm
- net GPIO0: track 0.00 -> 25.1 mm
- net GPIO15: track 0.00 -> 25.0 mm
- net GPIO14: track 0.00 -> 22.8 mm
- net GPIO12: track 0.00 -> 16.7 mm
- net RESET: track 0.00 -> 13.0 mm
- net Net-(R17-Pad2): track 0.00 -> 12.8 mm
- net GPIO13: track 0.00 -> 12.4 mm
- net Net-(J11-Pad1): track 0.00 -> 11.5 mm
- net Net-(J5-Pad1): track 0.00 -> 11.5 mm
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- added copper zone on B.Cu, net GND
- added copper zone on F.Cu, net GND
Other:
- board size 60 x 40 mm -> 71 x 57 mm
